Commit message: refactor: moved to gz_sim, changed resource path
Moved from Ignition gazebo to Gazebo Harmonic for better compatatibility
with PX4. Change resource path from IGN_GAZEBO_RESOURCE_PATH to
GZ_SIM_RESOURCE PATH inside launch files. Splited tarrot xacro into
multiple files to ensure DRY code

File: ros2_ws/src/uav/urdf/gazebo.xacro (robot description, xacro)
@@ -1,9 +1,6 @@
 <?xml version="1.0" encoding="UTF-8"?>
-<robot name="tarot" xmlns:xacro="https://www.ros.org/wiki/xacro">
+<robot name="tarot" xmlns:xacro="http://www.ros.org/wiki/xacro">
   <gazebo reference="base_link">
     <material>Gazebo/DarkGray</material>
-  </gazebo>
-  <gazebo reference="rotor_0">
-    <material>Gazebo/Red</material>
   </gazebo>
   <gazebo reference="rotor_1">
@@ -11,7 +8,10 @@
   </gazebo>
   <gazebo reference="rotor_2">
+    <material>Gazebo/Red</material>
+  </gazebo>
+  <gazebo reference="rotor_3">
     <material>Gazebo/Blue</material>
   </gazebo>
-  <gazebo reference="rotor_3">
+  <gazebo reference="rotor_4">
     <material>Gazebo/Blue</material>
   </gazebo>
@@ -21,4 +21,8 @@
       <real_time_factor>1</real_time_factor>
     </physics>
+    <plugin filename="ignition-gazebo-imu-system" name="ignition::gazebo::systems::Imu"></plugin>
+    <plugin filename="ignition-gazebo-sensors-system" name="ignition::gazebo::systems::Sensors">
+      <render_engine>ogre2</render_engine>
+    </plugin>
   </gazebo>
 </robot>

File: ros2_ws/src/uav/urdf/material.xacro (robot description, xacro)
@@ -1,4 +1,4 @@
 <?xml version="1.0" encoding="UTF-8"?>
-<robot name="trot" xmlns:xacro="https://www.ros.org/wiki/xacro">
+<robot name="trot" xmlns:xacro="http://www.ros.org/wiki/xacro">
   <material name="dark_gray">
     <color rgba="0.3 0.3 0.3 1.0"></color>

File: ros2_ws/src/uav/urdf/tarot.urdf.xacro (robot description, xacro)
@@ -1,6 +1,7 @@
 <?xml version="1.0" encoding="UTF-8"?>
-<robot name="tarot" xmlns:xacro="https://www.ros.org/wiki/xacro">
+<robot name="tarot" xmlns:xacro="http://www.ros.org/wiki/xacro">
   <xacro:include filename="$(find uav)/urdf/material.xacro"></xacro:include>
   <xacro:include filename="$(find uav)/urdf/gazebo.xacro"></xacro:include>
+  <xacro:include filename="$(find uav)/urdf/rotor.xacro"></xacro:include>
   <link name="base_link">
     <inertial>
@@ -20,128 +21,10 @@
         <mesh filename="package://uav/meshes/collision/tarot.stl" scale="0.00188 0.00183 0.00183"></mesh>
       </geometry>
-      <material name="dark_gray">
-        <color rgba="0.3 0.3 0.3 1.0"></color>
-      </material>
+      <material name="dark_gray"></material>
     </visual>
   </link>
-  <!-- Rotor 1 -->
-  <link name="rotor_1">
-    <inertial>
-      <origin rpy="0 0 0" xyz="0 0 0"></origin>
-      <mass value="0.005"></mass>
-      <inertia ixx="9.75e-07" ixy="0" ixz="0" iyy="0.000273104" iyz="0" izz="0.000274004"></inertia>
-    </inertial>
-    <collision>
-      <origin rpy="0 0 0" xyz="0 0 0"></origin>
-      <geometry>
-        <cylinder length="0.02" radius="0.32"></cylinder>
-      </geometry>
-    </collision>
-    <visual>
-      <origin rpy="0 0 0" xyz="-0.368 -0.362 -0.025"></origin>
-      <geometry>
-        <mesh filename="package://uav/meshes/collision/tarot_prop_ccw.stl" scale="2.5 2.5 1"></mesh>
-      </geometry>
-      <material name="red">
-        <color rgba="1.0 0 0 1.0"></color>
-      </material>
-    </visual>
-  </link>
-  <joint name="rotor_1_joint" type="continuous">
-    <parent link="base_link"></parent>
-    <child link="rotor_0"></child>
-    <origin rpy="0 0 0" xyz="0.40 -0.40 0.051"></origin>
-    <axis xyz="0 0 1"></axis>
-    <dynamics damping="0" friction="0"></dynamics>
-  </joint>
-  <!-- Rotor 2 -->
-  <link name="rotor_2">
-    <inertial>
-      <origin rpy="0 0 0" xyz="0 0 0"></origin>
-      <mass value="0.005"></mass>
-      <inertia ixx="9.75e-07" ixy="0" ixz="0" iyy="0.000273104" iyz="0" izz="0.000274004"></inertia>
-    </inertial>
-    <collision>
-      <origin rpy="0 0 0" xyz="0 0 0"></origin>
-      <geometry>
-        <cylinder length="0.02" radius="0.32"></cylinder>
-      </geometry>
-    </collision>
-    <visual>
-      <origin rpy="0 0 0" xyz="-0.368 -0.362 -0.025"></origin>
-      <geometry>
-        <mesh filename="package://uav/meshes/collision/tarot_prop_ccw.stl" scale="2.5 2.5 1"></mesh>
-      </geometry>
-      <material name="red">
-        <color rgba="1.0 0 0 1.0"></color>
-      </material>
-    </visual>
-  </link>
-  <joint name="rotor_2_joint" type="continuous">
-    <parent link="base_link"></parent>
-    <child link="rotor_1"></child>
-    <origin rpy="0 0 0" xyz="-0.40 0.40 0.051"></origin>
-    <axis xyz="0 0 1"></axis>
-    <dynamics damping="0.0" friction="0.0"></dynamics>
-  </joint>
-  <!-- Rotor 3 -->
-  <link name="rotor_3">
-    <inertial>
-      <origin rpy="0 0 0" xyz="0 0 0"></origin>
-      <mass value="0.005"></mass>
-      <inertia ixx="9.75e-07" ixy="0" ixz="0" iyy="0.000273104" iyz="0" izz="0.000274004"></inertia>
-    </inertial>
-    <collision>
-      <origin rpy="0 0 0" xyz="0 0 0"></origin>
-      <geometry>
-        <cylinder length="0.02" radius="0.32"></cylinder>
-      </geometry>
-    </collision>
-    <visual>
-      <origin rpy="0 0 0" xyz="-0.368 0.362 -0.025"></origin>
-      <geometry>
-        <mesh filename="package://uav/meshes/collision/tarot_prop_cw.stl" scale="2.5 2.5 1"></mesh>
-      </geometry>
-      <material name="blue">
-        <color rgba="0 0 1.0 1.0"></color>
-      </material>
-    </visual>
-  </link>
-  <joint name="rotor_3_joint" type="continuous">
-    <parent link="base_link"></parent>
-    <child link="rotor_2"></child>
-    <origin rpy="0 0 0" xyz="0.40 0.40 0.051"></origin>
-    <axis xyz="0 0 1"></axis>
-    <dynamics damping="0.0" friction="0.0"></dynamics>
-  </joint>
-  <!-- Rotor 4 -->
-  <link name="rotor_4">
-    <inertial>
-      <origin rpy="0 0 0" xyz="0 0 0"></origin>
-      <mass value="0.005"></mass>
-      <inertia ixx="9.75e-07" ixy="0" ixz="0" iyy="0.000273104" iyz="0" izz="0.000274004"></inertia>
-    </inertial>
-    <collision>
-      <origin rpy="0 0 0" xyz="0 0 0"></origin>
-      <geometry>
-        <cylinder length="0.02" radius="0.32"></cylinder>
-      </geometry>
-    </collision>
-    <visual>
-      <origin rpy="0 0 0" xyz="-0.368 0.362 -0.025"></origin>
-      <geometry>
-        <mesh filename="package://uav/meshes/collision/tarot_prop_cw.stl" scale="2.5 2.5 1"></mesh>
-      </geometry>
-      <material name="blue">
-        <color rgba="0 0 1.0 1.0"></color>
-      </material>
-    </visual>
-  </link>
-  <joint name="rotor_4_joint" type="continuous">
-    <parent link="base_link"></parent>
-    <child link="rotor_3"></child>
-    <origin rpy="0 0 0" xyz="-0.40 -0.40 0.051"></origin>
-    <axis xyz="0 0 1"></axis>
-    <dynamics damping="0" friction="0"></dynamics>
-  </joint>
+  <xacro:rotor number="1" rotation_type="ccw" xyz="0.40 -0.40 0.051"></xacro:rotor>
+  <xacro:rotor number="2" rotation_type="ccw" xyz="-0.40 0.40 0.051"></xacro:rotor>
+  <xacro:rotor number="3" rotation_type="cw" xyz="0.40 0.40 0.051"></xacro:rotor>
+  <xacro:rotor number="4" rotation_type="cw" xyz="-0.40 -0.40 0.051"></xacro:rotor>
 </robot>
