Commit message: refactor: migrate to gz_sim (harmonic)

File: ros2_ws/src/uav/urdf/rotor.xacro (robot description, xacro)
@@ -29,24 +29,24 @@
       <dynamics damping="0" friction="0"></dynamics>
     </joint>
-    <gazebo reference="motor_${number}">
-      <plugin filename="ignition-gazebo-multicopter-motor-model-system" name="ignition::gazebo::systems::MulticopterMotorModel">
-        <robotNamespace>tarot</robotNamespace>
-        <jointName>motor_${number}_joint</jointName>
-        <linkName>motor_${number}</linkName>
-        <turningDirection>${rotation_type}</turningDirection>
-        <timeConstantUp>0.0125</timeConstantUp>
-        <timeConstantDown>0.025</timeConstantDown>
-        <maxRotVelocity>1100</maxRotVelocity>
-        <motorConstant>8.54858e-06</motorConstant>
-        <momentConstant>0.06</momentConstant>
-        <commandSubTopic>command/motor_speed</commandSubTopic>
-        <motorNumber>${number}</motorNumber>
-        <rotorDragCoefficient>0.000175</rotorDragCoefficient>
-        <rollingMomentCoefficient>1e-06</rollingMomentCoefficient>
-        <motorSpeedPubTopic>motor_speed/${number}</motorSpeedPubTopic>
-        <rotorVelocitySlowdownSim>10</rotorVelocitySlowdownSim>
-        <motorType>velocity</motorType>
-      </plugin>
-    </gazebo>
+    <!-- <gazebo reference="motor_${number}"> -->
+    <!--   <plugin filename="ignition-gazebo-multicopter-motor-model-system" name="ignition::gazebo::systems::MulticopterMotorModel"> -->
+    <!--     <robotNamespace>tarot</robotNamespace> -->
+    <!--     <jointName>motor_${number}_joint</jointName> -->
+    <!--     <linkName>motor_${number}</linkName> -->
+    <!--     <turningDirection>${rotation_type}</turningDirection> -->
+    <!--     <timeConstantUp>0.0125</timeConstantUp> -->
+    <!--     <timeConstantDown>0.025</timeConstantDown> -->
+    <!--     <maxRotVelocity>1100</maxRotVelocity> -->
+    <!--     <motorConstant>8.54858e-06</motorConstant> -->
+    <!--     <momentConstant>0.06</momentConstant> -->
+    <!--     <commandSubTopic>command/motor_speed</commandSubTopic> -->
+    <!--     <motorNumber>${number}</motorNumber> -->
+    <!--     <rotorDragCoefficient>0.000175</rotorDragCoefficient> -->
+    <!--     <rollingMomentCoefficient>1e-06</rollingMomentCoefficient> -->
+    <!--     <motorSpeedPubTopic>motor_speed/${number}</motorSpeedPubTopic> -->
+    <!--     <rotorVelocitySlowdownSim>10</rotorVelocitySlowdownSim> -->
+    <!--     <motorType>velocity</motorType> -->
+    <!--   </plugin> -->
+    <!-- </gazebo> -->
   </xacro:macro>
 </robot>

File: ros2_ws/src/ugv/urdf/gazebo.xacro (robot description, xacro)
@@ -1,4 +1,4 @@
 <?xml version="1.0" encoding="UTF-8"?>
-<robot name="m2wr" xmlns:xacro="https://www.ros.org/wiki/xacro">
+<robot name="m2wr" xmlns:xacro="http://www.ros.org/wiki/xacro">
   <gazebo reference="motor_1">
     <material>Gazebo/Gray</material>
@@ -25,5 +25,4 @@
     <material>Gazebo/Gray</material>
   </gazebo>
-  <!--test them banh-->
   <gazebo reference="front_right_wheel_link">
     <material>Gazebo/Gray</material>
@@ -33,6 +32,13 @@
   </gazebo>
   <gazebo>
-    <plugin filename="libign_ros2_control-system.so" name="ign_ros2_control::IgnitionROS2ControlPlugin">
-      <parameters>$(find ugv)/config/controllers.yaml</parameters>
+    <plugin filename="gz-sim-mecanum-drive-system" name="gz::sim::systems::MecanumDrive">
+      <front_left_joint>front_left_wheel_joint</front_left_joint>
+      <front_right_joint>front_right_wheel_joint</front_right_joint>
+      <back_left_joint>rear_left_wheel_joint</back_left_joint>
+      <back_right_joint>rear_right_wheel_joint</back_right_joint>
+      <topic>/model/fuji_mecanum/cmd_vel</topic>
+    </plugin>
+    <plugin filename="gz-sim-joint-state-publisher-system" name="gz::sim::systems::JointStatePublisher">
+      <topic>/joint_states</topic>
     </plugin>
   </gazebo>

File: ros2_ws/src/ugv/urdf/joints.xacro (robot description, xacro)
@@ -1,4 +1,4 @@
 <?xml version="1.0" encoding="UTF-8"?>
-<robot xmlns:xacro="https://www.ros.org/wiki/xacro">
+<robot xmlns:xacro="http://www.ros.org/wiki/xacro">
   <xacro:macro name="joint" params="name type parent child xyz rpy">
     <joint name="${name}" type="${type}">

File: ros2_ws/src/ugv/urdf/material.xacro (robot description, xacro)
@@ -1,4 +1,4 @@
 <?xml version="1.0" encoding="UTF-8"?>
-<robot name="m2wr" xmlns:xacro="https://www.ros.org/wiki/xacro">
+<robot name="m2wr" xmlns:xacro="http://www.ros.org/wiki/xacro">
   <material name="black">
     <color rgba="0.0 0.0 0.0 1.0"></color>

File: ros2_ws/src/ugv/urdf/mecanum.xacro (robot description, xacro)
@@ -1,4 +1,4 @@
 <?xml version="1.0" encoding="UTF-8"?>
-<robot name="mecanum_wheel" xmlns:xacro="http://ros.org/wiki/xacro">
+<robot name="mecanum_wheel" xmlns:xacro="http://www.ros.org/wiki/xacro">
   <xacro:include filename="$(find ugv )/urdf/wheel.xacro"></xacro:include>
   <xacro:include filename="$(find ugv)/urdf/rollers.xacro"></xacro:include>

File: ros2_ws/src/ugv/urdf/rollers.xacro (robot description, xacro)
@@ -1,4 +1,4 @@
 <?xml version="1.0" encoding="UTF-8"?>
-<robot name="wheel" xmlns:xacro="https://www.ros.org/wiki/xacro">
+<robot name="wheel" xmlns:xacro="http://www.ros.org/wiki/xacro">
   <xacro:macro name="roller_origin" params="th side">
     <xacro:if value="${side==1}">

File: ros2_ws/src/ugv/urdf/shapes.xacro (robot description, xacro)
@@ -1,4 +1,4 @@
 <?xml version="1.0" encoding="UTF-8"?>
-<robot xmlns:xacro="https://www.ros.org/wiki/xacro">
+<robot xmlns:xacro="http://www.ros.org/wiki/xacro">
   <!-- Generic box link -->
   <xacro:macro name="box_link" params="name colli_name x y z mass color xyz rpy">

File: ros2_ws/src/ugv/urdf/ugv.urdf.xacro (robot description, xacro)
@@ -1,4 +1,4 @@
 <?xml version="1.0" encoding="UTF-8"?>
-<robot name="ugv" xmlns:xacro="https://ros.org/wiki/xacro">
+<robot name="ugv" xmlns:xacro="http://www.ros.org/wiki/xacro">
   <!-- Included files -->
   <xacro:include filename="$(find ugv)/urdf/mecanum.xacro"></xacro:include>
@@ -47,5 +47,5 @@
       <mass value="2.0"></mass>
       <origin rpy="0 0 0" xyz="0 0 0.0"></origin>
-      <inertia ixx="0.01" ixy="0" ixz="0" iyy="0.01" iyz="0" izz="0.01"></inertia>
+      <inertia ixx="0.007267" ixy="0" ixz="0" iyy="0.00195" iyz="0" izz="0.008017"></inertia>
     </inertial>
     <collision>
