Commit message: feat: add OS1 lidar, change docker image
adding new OS1-16 (testing) lidar to tarot drone model in Gazebo, bridge
to ROS2. change docker image to ros-humble-desktop to remove ignition
gazebo pre-installed in the other image

File: ros2_ws/src/tarot_description/urdf/gazebo.xacro (robot description, xacro)
@@ -36,50 +36,4 @@
       </magnetometer>
     </sensor>
-    <sensor name="imu_sensor" type="imu">
-      <always_on>1</always_on>
-      <update_rate>250</update_rate>
-      <imu>
-        <angular_velocity>
-          <x>
-            <noise type="gaussian">
-              <mean>0.0</mean>
-              <stddev>0.0008726646</stddev>
-            </noise>
-          </x>
-          <y>
-            <noise type="gaussian">
-              <mean>0.0</mean>
-              <stddev>0.0008726646</stddev>
-            </noise>
-          </y>
-          <z>
-            <noise type="gaussian">
-              <mean>0.0</mean>
-              <stddev>0.0008726646</stddev>
-            </noise>
-          </z>
-        </angular_velocity>
-        <linear_acceleration>
-          <x>
-            <noise type="gaussian">
-              <mean>0.0</mean>
-              <stddev>0.00637</stddev>
-            </noise>
-          </x>
-          <y>
-            <noise type="gaussian">
-              <mean>0.0</mean>
-              <stddev>0.00637</stddev>
-            </noise>
-          </y>
-          <z>
-            <noise type="gaussian">
-              <mean>0.0</mean>
-              <stddev>0.00686</stddev>
-            </noise>
-          </z>
-        </linear_acceleration>
-      </imu>
-    </sensor>
     <sensor name="navsat_sensor" type="navsat">
       <always_on>1</always_on>
@@ -100,6 +54,6 @@
   </gazebo>
   <gazebo>
-    <plugin filename="gz-sim-imu-system" name="gz::sim::systems::imu"></plugin>
-    <plugin filename="gz-sim-sensors-system" name="gz::sim::systems::sensors">
+    <plugin filename="gz-sim-imu-system" name="gz::sim::systems::Imu"></plugin>
+    <plugin filename="gz-sim-sensors-system" name="gz::sim::systems::Sensors">
       <render_engine>ogre2</render_engine>
     </plugin>

File: ros2_ws/src/tarot_description/urdf/tarot.urdf.xacro (robot description, xacro)
@@ -4,4 +4,5 @@
   <xacro:include filename="$(find tarot_description)/urdf/gazebo.xacro"></xacro:include>
   <xacro:include filename="$(find tarot_description)/urdf/rotor.xacro"></xacro:include>
+  <xacro:include filename="$(find tarot_description)/urdf/os_lidar.xacro"></xacro:include>
   <link name="base_link">
     <inertial>
@@ -24,4 +25,7 @@
     </visual>
   </link>
+  <xacro:os1 name="ouster" parent="base_link">
+    <origin rpy="0 0 0" xyz="0.013 0.025 0.51"></origin>
+  </xacro:os1>
   <xacro:rotor number="1" rotation_type="ccw" xyz="0.40 -0.38 0.501"></xacro:rotor>
   <xacro:rotor number="2" rotation_type="ccw" xyz="-0.40 0.41 0.501"></xacro:rotor>

Commit message: fix: fix lidar visual in rviz

File: ros2_ws/src/tarot_description/urdf/gazebo.xacro (robot description, xacro)
@@ -58,4 +58,10 @@
       <render_engine>ogre2</render_engine>
     </plugin>
+    <plugin filename="gz-sim-joint-state-publisher-system" name="gz::sim::systems::JointStatePublisher">
+      <joint_name>motor_1_joint</joint_name>
+      <joint_name>motor_2_joint</joint_name>
+      <joint_name>motor_3_joint</joint_name>
+      <joint_name>motor_4_joint</joint_name>
+    </plugin>
   </gazebo>
 </robot>

File: ros2_ws/src/tarot_description/urdf/os_lidar.xacro (robot description, xacro)
@@ -30,10 +30,10 @@
     <link name="${lidar_link}"></link>
     <joint name="${name}_imu_joint" type="fixed">
-      <parent link="${name}"></parent>
+      <parent link="${parent}"></parent>
       <child link="${imu_link}"></child>
       <origin rpy="0 0 0" xyz="0.006253 -0.011775 0.007645"></origin>
     </joint>
     <joint name="${name}_lidar_joint" type="fixed">
-      <parent link="${name}"></parent>
+      <parent link="${parent}"></parent>
       <child link="${lidar_link}"></child>
       <origin rpy="0 0 0" xyz="0.0 0.0 0.03618"></origin>
@@ -42,4 +42,5 @@
       <sensor name="${name}_lidar" type="gpu_lidar">
         <pose relative_to="${name}">0 0 0 0 0 0</pose>
+        <gz_frame_id>${lidar_link}</gz_frame_id>
         <visualize>false</visualize>
         <update_rate>${hz}</update_rate>
@@ -49,5 +50,5 @@
           <scan>
             <horizontal>
-              <samples>16</samples>
+              <samples>1024</samples>
               <resolution>1</resolution>
               <min_angle>${min_angle}</min_angle>
@@ -55,5 +56,5 @@
             </horizontal>
             <vertical>
-              <samples>10</samples>
+              <samples>16</samples>
               <resolution>1</resolution>
               <min_angle>${vfov_min}</min_angle>

File: ros2_ws/src/tarot_description/urdf/tarot.urdf.xacro (robot description, xacro)
@@ -12,5 +12,5 @@
     </inertial>
     <collision>
-      <origin rpy="1.5708 0 1.5697" xyz="0 0 0.45"></origin>
+      <origin rpy="1.5708 0 1.5697" xyz="0 0 0.95"></origin>
       <geometry>
         <mesh filename="package://tarot_description/models/tarot/meshes/collision/tarot.stl" scale="0.00188 0.00183 0.00183"></mesh>
@@ -18,5 +18,5 @@
     </collision>
     <visual>
-      <origin rpy="1.5708 0 1.5697" xyz="0 0 0.45"></origin>
+      <origin rpy="1.5708 0 1.5697" xyz="0 0 0.95"></origin>
       <geometry>
         <mesh filename="package://tarot_description/models/tarot/meshes/collision/tarot.stl" scale="0.00188 0.00183 0.00183"></mesh>
@@ -26,9 +26,9 @@
   </link>
   <xacro:os1 name="ouster" parent="base_link">
-    <origin rpy="0 0 0" xyz="0.013 0.025 0.51"></origin>
+    <origin rpy="0 0 0" xyz="0.013 0.025 1.01"></origin>
   </xacro:os1>
-  <xacro:rotor number="1" rotation_type="ccw" xyz="0.40 -0.38 0.501"></xacro:rotor>
-  <xacro:rotor number="2" rotation_type="ccw" xyz="-0.40 0.41 0.501"></xacro:rotor>
-  <xacro:rotor number="3" rotation_type="cw" xyz="0.40 0.40 0.501"></xacro:rotor>
-  <xacro:rotor number="4" rotation_type="cw" xyz="-0.40 -0.40 0.501"></xacro:rotor>
+  <xacro:rotor number="1" rotation_type="ccw" xyz="0.40 -0.38 1.001"></xacro:rotor>
+  <xacro:rotor number="2" rotation_type="ccw" xyz="-0.40 0.41 1.001"></xacro:rotor>
+  <xacro:rotor number="3" rotation_type="cw" xyz="0.40 0.40 1.001"></xacro:rotor>
+  <xacro:rotor number="4" rotation_type="cw" xyz="-0.40 -0.40 1.001"></xacro:rotor>
 </robot>

Commit message: fix: fix sdf for px4_sitl

File: ros2_ws/src/tarot_description/urdf/gazebo.xacro (robot description, xacro)
@@ -36,4 +36,51 @@
       </magnetometer>
     </sensor>
+    <sensor name="imu_sensor" type="imu">
+      <gz_frame_id>base_link</gz_frame_id>
+      <always_on>1</always_on>
+      <update_rate>250</update_rate>
+      <imu>
+        <angular_velocity>
+          <x>
+            <noise type="gaussian">
+              <mean>0.0</mean>
+              <stddev>0.0008726646</stddev>
+            </noise>
+          </x>
+          <y>
+            <noise type="gaussian">
+              <mean>0.0</mean>
+              <stddev>0.0008726646</stddev>
+            </noise>
+          </y>
+          <z>
+            <noise type="gaussian">
+              <mean>0.0</mean>
+              <stddev>0.0008726646</stddev>
+            </noise>
+          </z>
+        </angular_velocity>
+        <linear_acceleration>
+          <x>
+            <noise type="gaussian">
+              <mean>0.0</mean>
+              <stddev>0.00637</stddev>
+            </noise>
+          </x>
+          <y>
+            <noise type="gaussian">
+              <mean>0.0</mean>
+              <stddev>0.00637</stddev>
+            </noise>
+          </y>
+          <z>
+            <noise type="gaussian">
+              <mean>0.0</mean>
+              <stddev>0.00686</stddev>
+            </noise>
+          </z>
+        </linear_acceleration>
+      </imu>
+    </sensor>
     <sensor name="navsat_sensor" type="navsat">
       <always_on>1</always_on>
@@ -54,13 +101,75 @@
   </gazebo>
   <gazebo>
-    <plugin filename="gz-sim-imu-system" name="gz::sim::systems::Imu"></plugin>
-    <plugin filename="gz-sim-sensors-system" name="gz::sim::systems::Sensors">
-      <render_engine>ogre2</render_engine>
-    </plugin>
     <plugin filename="gz-sim-joint-state-publisher-system" name="gz::sim::systems::JointStatePublisher">
+      <joint_name>motor_0_joint</joint_name>
       <joint_name>motor_1_joint</joint_name>
       <joint_name>motor_2_joint</joint_name>
       <joint_name>motor_3_joint</joint_name>
-      <joint_name>motor_4_joint</joint_name>
+    </plugin>
+  </gazebo>
+  <gazebo>
+    <plugin filename="gz-sim-multicopter-motor-model-system" name="gz::sim::systems::MulticopterMotorModel">
+      <jointName>motor_0_joint</jointName>
+      <linkName>motor_0</linkName>
+      <turningDirection>ccw</turningDirection>
+      <timeConstantUp>0.0125</timeConstantUp>
+      <timeConstantDown>0.025</timeConstantDown>
+      <maxRotVelocity>1000.0</maxRotVelocity>
+      <motorConstant>8.54858e-06</motorConstant>
+      <momentConstant>0.016</momentConstant>
+      <commandSubTopic>command/motor_speed</commandSubTopic>
+      <motorNumber>0</motorNumber>
+      <rotorDragCoefficient>8.06428e-05</rotorDragCoefficient>
+      <rollingMomentCoefficient>1e-06</rollingMomentCoefficient>
+      <rotorVelocitySlowdownSim>10</rotorVelocitySlowdownSim>
+      <motorType>velocity</motorType>
+    </plugin>
+    <plugin filename="gz-sim-multicopter-motor-model-system" name="gz::sim::systems::MulticopterMotorModel">
+      <jointName>motor_1_joint</jointName>
+      <linkName>motor_1</linkName>
+      <turningDirection>ccw</turningDirection>
+      <timeConstantUp>0.0125</timeConstantUp>
+      <timeConstantDown>0.025</timeConstantDown>
+      <maxRotVelocity>1000.0</maxRotVelocity>
+      <motorConstant>8.54858e-06</motorConstant>
+      <momentConstant>0.016</momentConstant>
+      <commandSubTopic>command/motor_speed</commandSubTopic>
+      <motorNumber>1</motorNumber>
+      <rotorDragCoefficient>8.06428e-05</rotorDragCoefficient>
+      <rollingMomentCoefficient>1e-06</rollingMomentCoefficient>
+      <rotorVelocitySlowdownSim>10</rotorVelocitySlowdownSim>
+      <motorType>velocity</motorType>
+    </plugin>
+    <plugin filename="gz-sim-multicopter-motor-model-system" name="gz::sim::systems::MulticopterMotorModel">
+      <jointName>motor_2_joint</jointName>
+      <linkName>motor_2</linkName>
+      <turningDirection>cw</turningDirection>
+      <timeConstantUp>0.0125</timeConstantUp>
+      <timeConstantDown>0.025</timeConstantDown>
+      <maxRotVelocity>1000.0</maxRotVelocity>
+      <motorConstant>8.54858e-06</motorConstant>
+      <momentConstant>0.016</momentConstant>
+      <commandSubTopic>command/motor_speed</commandSubTopic>
+      <motorNumber>2</motorNumber>
+      <rotorDragCoefficient>8.06428e-05</rotorDragCoefficient>
+      <rollingMomentCoefficient>1e-06</rollingMomentCoefficient>
+      <rotorVelocitySlowdownSim>10</rotorVelocitySlowdownSim>
+      <motorType>velocity</motorType>
+    </plugin>
+    <plugin filename="gz-sim-multicopter-motor-model-system" name="gz::sim::systems::MulticopterMotorModel">
+      <jointName>motor_3_joint</jointName>
+      <linkName>motor_3</linkName>
+      <turningDirection>cw</turningDirection>
+      <timeConstantUp>0.0125</timeConstantUp>
+      <timeConstantDown>0.025</timeConstantDown>
+      <maxRotVelocity>1000.0</maxRotVelocity>
+      <motorConstant>8.54858e-06</motorConstant>
+      <momentConstant>0.016</momentConstant>
+      <commandSubTopic>command/motor_speed</commandSubTopic>
+      <motorNumber>3</motorNumber>
+      <rotorDragCoefficient>8.06428e-05</rotorDragCoefficient>
+      <rollingMomentCoefficient>1e-06</rollingMomentCoefficient>
+      <rotorVelocitySlowdownSim>10</rotorVelocitySlowdownSim>
+      <motorType>velocity</motorType>
     </plugin>
   </gazebo>

File: ros2_ws/src/tarot_description/urdf/os_lidar.xacro (robot description, xacro)
@@ -14,5 +14,5 @@
         <inertia ixx="0.000241148" ixy="0" ixz="0" iyy="0.000241148" iyz="0" izz="0.000264"></inertia>
       </inertial>
-      <collision name="base_collision">
+      <collision name="${name}_collision">
         <origin rpy="0 0 0" xyz="0 0 0.0365"></origin>
         <geometry>
@@ -20,5 +20,5 @@
         </geometry>
       </collision>
-      <visual name="base_visual">
+      <visual name="${name}_visual">
         <origin rpy="0 0 1.5707" xyz="0 0 0.0"></origin>
         <geometry>
@@ -30,10 +30,10 @@
     <link name="${lidar_link}"></link>
     <joint name="${name}_imu_joint" type="fixed">
-      <parent link="${parent}"></parent>
+      <parent link="${name}"></parent>
       <child link="${imu_link}"></child>
       <origin rpy="0 0 0" xyz="0.006253 -0.011775 0.007645"></origin>
     </joint>
     <joint name="${name}_lidar_joint" type="fixed">
-      <parent link="${parent}"></parent>
+      <parent link="${name}"></parent>
       <child link="${lidar_link}"></child>
       <origin rpy="0 0 0" xyz="0.0 0.0 0.03618"></origin>

File: ros2_ws/src/tarot_description/urdf/rotor.xacro (robot description, xacro)
@@ -29,22 +29,4 @@
       <dynamics damping="0" friction="0"></dynamics>
     </joint>
-    <gazebo reference="motor_${number}">
-      <plugin filename="gz-sim-multicopter-motor-model-system" name="gz::sim::systems::MulticopterMotorModel">
-        <jointName>motor_${number}_joint</jointName>
-        <linkName>motor_${number}</linkName>
-        <turningDirection>${rotation_type}</turningDirection>
-        <timeConstantUp>0.0125</timeConstantUp>
-        <timeConstantDown>0.025</timeConstantDown>
-        <maxRotVelocity>1000</maxRotVelocity>
-        <motorConstant>8.54858e-06</motorConstant>
-        <momentConstant>0.06</momentConstant>
-        <commandSubTopic>command/motor_speed</commandSubTopic>
-        <motorNumber>${number}</motorNumber>
-        <rotorDragCoefficient>0.000175</rotorDragCoefficient>
-        <rollingMomentCoefficient>1e-06</rollingMomentCoefficient>
-        <rotorVelocitySlowdownSim>10</rotorVelocitySlowdownSim>
-        <motorType>velocity</motorType>
-      </plugin>
-    </gazebo>
   </xacro:macro>
 </robot>

File: ros2_ws/src/tarot_description/urdf/tarot.urdf.xacro (robot description, xacro)
@@ -12,5 +12,5 @@
     </inertial>
     <collision>
-      <origin rpy="1.5708 0 1.5697" xyz="0 0 0.95"></origin>
+      <origin rpy="1.5708 0 1.5697" xyz="0 0 0.45"></origin>
       <geometry>
         <mesh filename="package://tarot_description/models/tarot/meshes/collision/tarot.stl" scale="0.00188 0.00183 0.00183"></mesh>
@@ -18,5 +18,5 @@
     </collision>
     <visual>
-      <origin rpy="1.5708 0 1.5697" xyz="0 0 0.95"></origin>
+      <origin rpy="1.5708 0 1.5697" xyz="0 0 0.45"></origin>
       <geometry>
         <mesh filename="package://tarot_description/models/tarot/meshes/collision/tarot.stl" scale="0.00188 0.00183 0.00183"></mesh>
@@ -26,9 +26,9 @@
   </link>
   <xacro:os1 name="ouster" parent="base_link">
-    <origin rpy="0 0 0" xyz="0.013 0.025 1.01"></origin>
+    <origin rpy="0 0 0" xyz="0.013 0.025 0.51"></origin>
   </xacro:os1>
-  <xacro:rotor number="1" rotation_type="ccw" xyz="0.40 -0.38 1.001"></xacro:rotor>
-  <xacro:rotor number="2" rotation_type="ccw" xyz="-0.40 0.41 1.001"></xacro:rotor>
-  <xacro:rotor number="3" rotation_type="cw" xyz="0.40 0.40 1.001"></xacro:rotor>
-  <xacro:rotor number="4" rotation_type="cw" xyz="-0.40 -0.40 1.001"></xacro:rotor>
+  <xacro:rotor number="0" rotation_type="ccw" xyz="0.40 -0.38 0.501"></xacro:rotor>
+  <xacro:rotor number="1" rotation_type="ccw" xyz="-0.40 0.41 0.501"></xacro:rotor>
+  <xacro:rotor number="2" rotation_type="cw" xyz="0.40 0.40 0.501"></xacro:rotor>
+  <xacro:rotor number="3" rotation_type="cw" xyz="-0.40 -0.40 0.501"></xacro:rotor>
 </robot>
